File: hardware/TMC2209_Driver.kicad_pcb (KiCad board)
At the start: 2 copper layers, 36.7 x 39.4 mm, 31 parts, among them J1 PCIe_Stepper, J2 Conn_01x04_Male, U1 TMC2209-LA, U2 74LVC1G06, U3 24LC02

Commit message: 2209 rotated version
Parts:
- removed FID1, FID2, FID3, FID4: Fiducial, PrntrBoardV2:Fiducial_1mm_Dia_2.54mm_Outer_CopperTop
- moved C15 27.2 mm to (128.5, 78.0), turned to 180 degrees
- moved C11 24.3 mm to (142.6, 80.9), turned to -90 degrees
- moved C12 22.5 mm to (141.0, 80.8), turned to -90 degrees
- moved C7 22.0 mm to (135.6, 79.1), turned to 0 degrees
- moved C9 21.0 mm to (142.6, 96.9), turned to 90 degrees
- moved C10 19.0 mm to (141.1, 96.9), turned to 90 degrees
- moved J2 18.1 mm to (141.6, 88.9), turned to 90 degrees
- moved R3 16.2 mm to (136.8, 82.9), turned to -90 degrees
- moved C8 12.7 mm to (135.0, 98.3)
- moved R2 12.3 mm to (136.9, 94.8), turned to 90 degrees
- moved C4 11.9 mm to (127.3, 83.0), turned to -90 degrees
- moved C3 11.7 mm to (128.9, 83.0), turned to -90 degrees
- moved C6 11.4 mm to (133.0, 84.2), turned to 90 degrees
- moved C2 11.3 mm to (124.7, 84.4), turned to -90 degrees
- moved JP1 7.20 mm to (123.9, 92.1), turned to 180 degrees
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Connections:
- J1 pad : (no net) -> /ID_0
Routing:
- net /V_MOTORS: track 103.3 -> 55.4 mm
- net /~ENABLE: track 26.8 -> 44.8 mm, vias 2 -> 4
- net /STEP: track 43.9 -> 28.3 mm, vias 4 -> 3
- net /ID_1: track 44.4 -> 56.2 mm, vias 4 -> 3
- net /ID_0: track 47.8 -> 59.1 mm, vias 3 -> 4
- net /DIR: track 41.1 -> 30.2 mm, vias 4 -> 2
- net /DIAG: track 15.5 -> 22.9 mm, vias 2 -> 0
- net /ID_2: track 34.6 -> 29.9 mm
- net VCC: track 44.4 -> 40.5 mm, vias 7 -> 5
- net GND: track 52.4 -> 54.5 mm, vias 40 -> 68
- net /CLOCK: track 17.6 -> 19.6 mm, vias 5 -> 1
- net /SDA: track 18.9 -> 17.2 mm
- net /RX: track 23.1 -> 24.8 mm, vias 3 -> 1
- net /SCL: track 18.1 -> 19.1 mm
- net /MOTB2: track 3.66 -> 2.87 mm
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Other:
- board text added: "CLK"
- board text added: "Ext Int"
- board text removed: "*"
- board text removed: "1-2 Int Clk 2-3 Ext Clk"
