File: hardware/TMC2209_Driver.kicad_sch (KiCad schematic)
At the start: 31 parts, among them J1 PCIe_Stepper, J2 Conn_01x04_Male, U1 TMC2209-LA, U2 74LVC1G06, U3 24LC02

Commit message: 2209 rotated version
Parts:
- removed FID1, FID2, FID3, FID4: Fiducial, PrntrBoardV2:Fiducial_1mm_Dia_2.54mm_Outer_CopperTop, symbol Mechanical:Fiducial
Changed lines of the file:
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@@
   (junction (at 254 91.44) (diameter 1.016) (color 0 0 0 0))
   (junction (at 254 93.98) (diameter 1.016) (color 0 0 0 0))
+  (no_connect (at 101.6 88.9))
   (no_connect (at 101.6 99.06))
   (no_connect (at 120.65 68.58))
-  (no_connect (at 101.6 88.9))
   (wire (pts (xy 71.755 93.98) (xy 59.055 93.98))
     (stroke (width 0) (type solid) (color 0 0 0 0))
@@
     )
     (property "Datasheet" "" (id 3) (at 254 98.425 0)
-      (effects (font (size 1.27 1.27)) hide)
-    )
-  )
-  (symbol (lib_id "Mechanical:Fiducial") (at 26.67 114.3 0) (unit 1)
-    (in_bom no) (on_board yes)
-    (property "Reference" "FID1" (id 0) (at 28.829 113.1316 0)
-      (effects (font (size 1.27 1.27)) (justify left))
-    )
-    (property "Value" "Fiducial" (id 1) (at 28.829 115.443 0)
-      (effects (font (size 1.27 1.27)) (justify left))
-    )
-    (property "Footprint" "PrntrBoardV2:Fiducial_1mm_Dia_2.54mm_Outer_CopperTop" (id 2) (at 26.67 114.3 0)
-      (effects (font (size 1.27 1.27)) hide)
-    )
-    (property "Datasheet" "~" (id 3) (at 26.67 114.3 0)
-      (effects (font (size 1.27 1.27)) hide)
-    )
-  )
-  (symbol (lib_id "Mechanical:Fiducial") (at 26.67 123.19 0) (unit 1)
-    (in_bom no) (on_board yes)
-    (property "Reference" "FID2" (id 0) (at 28.829 122.0216 0)
-      (effects (font (size 1.27 1.27)) (justify left))
-    )
-    (property "Value" "Fiducial" (id 1) (at 28.829 124.333 0)
-      (effects (font (size 1.27 1.27)) (justify left))
-    )
-    (property "Footprint" "PrntrBoardV2:Fiducial_1mm_Dia_2.54mm_Outer_CopperTop" (id 2) (at 26.67 123.19 0)
-      (effects (font (size 1.27 1.27)) hide)
-    )
-    (property "Datasheet" "~" (id 3) (at 26.67 123.19 0)
-      (effects (font (size 1.27 1.27)) hide)
-    )
-  )
-  (symbol (lib_id "Mechanical:Fiducial") (at 26.67 130.81 0) (unit 1)
-    (in_bom no) (on_board yes)
-    (property "Reference" "FID3" (id 0) (at 28.829 129.6416 0)
-      (effects (font (size 1.27 1.27)) (justify left))
-    )
-    (property "Value" "Fiducial" (id 1) (at 28.829 131.953 0)
-      (effects (font (size 1.27 1.27)) (justify left))
-    )
-    (property "Footprint" "PrntrBoardV2:Fiducial_1mm_Dia_2.54mm_Outer_CopperTop" (id 2) (at 26.67 130.81 0)
-      (effects (font (size 1.27 1.27)) hide)
-    )
-    (property "Datasheet" "~" (id 3) (at 26.67 130.81 0)
-      (effects (font (size 1.27 1.27)) hide)
-    )
-  )
-  (symbol (lib_id "Mechanical:Fiducial") (at 26.67 137.795 0) (unit 1)
-    (in_bom no) (on_board yes)
-    (property "Reference" "FID4" (id 0) (at 28.829 136.6266 0)
-      (effects (font (size 1.27 1.27)) (justify left))
-    )
-    (property "Value" "Fiducial" (id 1) (at 28.829 138.938 0)
-      (effects (font (size 1.27 1.27)) (justify left))
-    )
-    (property "Footprint" "PrntrBoardV2:Fiducial_1mm_Dia_2.54mm_Outer_CopperTop" (id 2) (at 26.67 137.795 0)
-      (effects (font (size 1.27 1.27)) hide)
-    )
-    (property "Datasheet" "~" (id 3) (at 26.67 137.795 0)
       (effects (font (size 1.27 1.27)) hide)
     )
@@
       (reference "C15") (unit 1) (value "100uV 35V") (footprint "Capacitor_SMD:CP_Elec_6.3x7.7")
     )
-    (path "/00000000-0000-0000-0000-00005d9a69ec"
-      (reference "FID1") (unit 1) (value "Fiducial") (footprint "PrntrBoardV2:Fiducial_1mm_Dia_2.54mm_Outer_CopperTop")
-    )
-    (path "/00000000-0000-0000-0000-00005d9a69ed"
-      (reference "FID2") (unit 1) (value "Fiducial") (footprint "PrntrBoardV2:Fiducial_1mm_Dia_2.54mm_Outer_CopperTop")
-    )
-    (path "/00000000-0000-0000-0000-00005d9a69ee"
-      (reference "FID3") (unit 1) (value "Fiducial") (footprint "PrntrBoardV2:Fiducial_1mm_Dia_2.54mm_Outer_CopperTop")
-    )
-    (path "/00000000-0000-0000-0000-00005d9a69ef"
-      (reference "FID4") (unit 1) (value "Fiducial") (footprint "PrntrBoardV2:Fiducial_1mm_Dia_2.54mm_Outer_CopperTop")
-    )
     (path "/00000000-0000-0000-0000-00005d9a69f2"
