File: hardware/Endstops.kicad_sch (KiCad schematic)
At the start: 47 parts

Commit message: Intermediate checkin
Parts:
- C33, C34, C35, C36, C37, C38, C39, C40: footprint PrntrBoardV2:C_0603_1608Metric -> Capacitor_SMD:C_0402_1005Metric; LCSC Part # C1588 -> C1523; Part # CL10B102KB8NNNC -> 0402B102K500NT
- R29, R30, R31, R35, R36, R37, R41, R42: footprint PrntrBoardV2:R_0603_1608Metric -> Resistor_SMD:R_0402_1005Metric; LCSC Part # C21190 -> C11702; Part # 0603WAF1001T5E -> 0402WGF1001TCE
- R32, R33, R34, R38, R39, R40, R43, R44, R47: footprint PrntrBoardV2:R_0603_1608Metric -> Resistor_SMD:R_0402_1005Metric; LCSC Part # C25804 -> C25744; Part # 0603WAF1002T5E -> 0402WGF1002TCE
