File: hardware/Power.kicad_sch (KiCad schematic)
At the start: 34 parts, among them J1 JST XH, J2 JST XH, J22 JST XH, J23 JST XH, J24 JST XH, J25 JST XH, J26 JST XH, J27 JST XH, J28 KF350, Q1 NCE40P40K, U4 AMS1117-3.3, U5 DCBuck

Commit message: Intermediate checkin
Parts:
- removed C20, C23, C26: 10uF, PrntrBoardV2:C_0603_1608Metric, symbol Device:C
- removed C21, C22: 0.1uF, PrntrBoardV2:C_0603_1608Metric, symbol Device:C
- removed J28: KF350, PrntrBoardV2:TerminalBlock_Phoenix_PT-1,5-2-3.5-H_1x02_P3.50mm_Horizontal, symbol Connector:Screw_Terminal_01x02
- removed U4: AMS1117-3.3, Package_TO_SOT_SMD:SOT-223-3_TabPin2, symbol Regulator_Linear:AMS1117-3.3
- removed U5: DCBuck, PrntrBoardV2:Buck2217, symbol BuckConverter:DCBuck
- R13, R14: footprint PrntrBoardV2:R_0603_1608Metric -> Resistor_SMD:R_0402_1005Metric; LCSC Part # C25804 -> C25744; Part # 0603WAF1002T5E -> 0402WGF1002TCE
- R15: footprint PrntrBoardV2:R_0603_1608Metric -> Resistor_SMD:R_0402_1005Metric; LCSC Part # C23179 -> C25117; Part # 0603WAF4700T5E -> 0402WGF4700TCE
- R16: footprint PrntrBoardV2:R_0603_1608Metric -> Resistor_SMD:R_0402_1005Metric; LCSC Part # C21190 -> C11702; Part # 0603WAF1001T5E -> 0402WGF1001TCE
- R71: footprint PrntrBoardV2:R_0603_1608Metric -> Resistor_SMD:R_0402_1005Metric; LCSC Part # C25803 -> C25741; Part # 0603WAF1003T5E -> 0402WGF1003TCE
Connections:
- net Vin: now reaches F2.1, F3.1, F4.1, J_power_in1.2 (Pin_2)
Other:
- moved on the sheet: C24, C25, D2, D3, D4, D5, D6, F2, F3, F4, J1, J2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
