File: hardware/PrntrBoardV3.kicad_sch (KiCad schematic)
At the start: 16 parts, among them J28 JST XH, U1001 TPS5430DDA

Commit message: V3 added
Parts:
- removed C1001: 10n, Capacitor_SMD:C_0402_1005Metric, symbol Device:C
- removed C1002, C1003: 10u/30V, Capacitor_SMD:C_2220_5650Metric, symbol Device:C
- removed C1004: 220u/25V, Capacitor_THT:CP_Radial_D6.3mm_P2.50mm, symbol Device:CP
- removed D1001: SS54, Diode_SMD:D_SMA, symbol Device:D_Schottky
- removed J28: JST XH, Connector_JST:JST_XH_B2B-XH-A_1x02_P2.50mm_Vertical, symbol Connector_Generic:Conn_02x01
- removed JM1: Conn_02x25_Counter_Clockwise, Connector_IDC:IDC-Header_2x25_P2.54mm_Vertical, symbol Connector_Generic:Conn_02x25_Odd_Even
- removed JP1: Jumper_3_Open, Connector_PinHeader_2.54mm:PinHeader_1x03_P2.54mm_Vertical, symbol Jumper:Jumper_3_Open
- removed L1001: 22u/4A, Inductor_THT:L_Radial_D9.5mm_P5.00mm_Fastron_07HVP, symbol Device:L_Core_Iron
- removed R1001: 10k/1%, Resistor_SMD:R_0402_1005Metric, symbol Device:R
- removed R1002: 3k24/1%, Resistor_SMD:R_0402_1005Metric, symbol Device:R
- removed U1001: TPS5430DDA, Package_SO:TI_SO-PowerPAD-8_ThermalVias, symbol Regulator_Switching:TPS5430DDA
- added G1: LION_LOGO, PrntrBoardV2:lion_logo_big, symbol lion_logo:LION_LOGO
- added LOGO1: Logo_Open_Hardware_Small, Symbol:OSHW-Logo_7.5x8mm_SilkScreen, symbol Graphic:Logo_Open_Hardware_Small
- H1, H2, H3, H4: now left out of the parts list
Connections:
- no-connect marks 1 -> 0
Other:
- sheet ADC: file Adc.kicad_sch -> AdcV3.kicad_sch
- sheet End Stops: file Endstops.kicad_sch -> EndstopsV3.kicad_sch
- sheet IO: file IO_Connectors.kicad_sch -> IO_ConnectorsV3.kicad_sch
- sheet MCU: file mcu_144.kicad_sch -> McuV3.kicad_sch
- sheet PWM: file Pwm.kicad_sch -> PwmV3.kicad_sch
- sheet Power: file Power.kicad_sch -> PowerV3.kicad_sch
- note removed: "1.221V"
- note removed: "8 PORT PCIex Expander"
- note removed: "EXTERNAL POWER"
- note removed: "Input 24V, 50W"
- note removed: "Output +5VA / 3A (4A in peak)"
